Commit message: started building real sense camera class and fixed bugs. Building infrastructure for camera localization. Also fixed bugs in transforms and using camera optical depth frame as the camera frame

File: src/deps/abb/abb_irb2600_support/urdf/irb2600_12_165.xacro (robot description, xacro)
@@ -3,3 +3,10 @@
   <xacro:include filename="$(find abb_irb2600_support)/urdf/irb2600_12_165_macro.xacro"/>
   <xacro:abb_irb2600_12_165 prefix=""/>
+  <xacro:arg name="use_nominal_extrinsics" default="true" />
+  <xacro:arg name="add_plug" default="true" />
+  <xacro:arg name="use_mesh" default="true" />
+  <xacro:include filename="$(find realsense2_description)/urdf/_d415.urdf.xacro" />
+  <xacro:sensor_d415 parent="camera_mount" use_nominal_extrinsics="$(arg use_nominal_extrinsics)" add_plug="$(arg add_plug)" use_mesh="$(arg use_mesh)">
+    <origin xyz="-0.004 0.0 0.032" rpy="0 -1.57 0"/>
+  </xacro:sensor_d415>
 </robot>

File: src/deps/abb/abb_irb2600_support/urdf/irb2600_12_165_macro.xacro (robot description, xacro)
@@ -175,26 +175,20 @@
       <child link="${prefix}tool0" />
     </joint>
-    <!-- Camera -->
     <link name="camera_mount">
-    <visual>
-        <geometry>
-            <mesh filename="package://system/database/meshes/camera_mount.stl"
-                scale="1 1 1"/>
-        </geometry>
-        <material name="ABS" >
-            <color rgba="0.5 0.5 0.5 1.0" />
-            </material>
-        </visual>
-    </link>
-    <link name="camera_base">
-    <visual>
-        <geometry>
-            <mesh filename="package://system/database/meshes/d415.stl"
-                scale="1 1 1"/>
-        </geometry>
-        <material name="ABS" >
-            <color rgba="0.5 0.5 0.5 1.0" />
-            </material>
-        </visual>
+      <visual>
+      <geometry>
+          <mesh filename="package://system/database/meshes/camera_mount.stl"
+              scale="1 1 1"/>
+      </geometry>
+      <material name="ABS" >
+          <color rgba="0.5 0.5 0.5 1.0" />
+          </material>
+      </visual>
+      <collision>
+        <origin xyz="0 0 0" rpy="0 0 0" />
+        <geometry>
+          <mesh filename="package://system/database/meshes/camera_mount.stl" />
+        </geometry>
+      </collision>
     </link>
     <joint type="fixed" name="mount_joint">
@@ -203,9 +197,4 @@
         <child link="camera_mount"/>
     </joint>
-    <joint type="fixed" name="camera_joint">
-        <origin xyz="-0.0145 0 0.0385" rpy="0 0 1.57"/>
-        <parent link="camera_mount"/>
-        <child link="camera_base"/>
-    </joint>
   </xacro:macro>
 </robot>

Commit message: Updated collision plane positions, launch file for robot ip, and robot home location based on real world setup

File: src/deps/abb/abb_irb2600_support/urdf/irb2600_12_165.xacro (robot description, xacro)
@@ -8,5 +8,5 @@
   <xacro:include filename="$(find realsense2_description)/urdf/_d415.urdf.xacro" />
   <xacro:sensor_d415 parent="camera_mount" use_nominal_extrinsics="$(arg use_nominal_extrinsics)" add_plug="$(arg add_plug)" use_mesh="$(arg use_mesh)">
-    <origin xyz="-0.004 0.0 0.032" rpy="0 -1.57 0"/>
+    <origin xyz="-0.004 0.0 0.031" rpy="0 -1.57 0"/>
   </xacro:sensor_d415>
 </robot>
