Commit message: All parts working

File: src/deps/abb/abb_irb2600_support/urdf/irb2600_12_165_macro copy.xacro (robot description, xacro)
@@ -138,5 +138,5 @@
       <child link="${prefix}link_4" />
       <axis xyz="1 0 0" />
-      <limit lower="-1.8" upper="5.23" effort="0" velocity="6.283" />
+      <limit lower="-6.981" upper="6.981" effort="0" velocity="6.283" />
     </joint>
     <joint name="${prefix}joint_5" type="revolute">
