Commit message: pointcloud visualization for simulated camera added. Will need to fix some issues. Visible cloud is not updating as desired

File: src/deps/abb/abb_irb2600_support/urdf/irb2600_12_165_macro.xacro (robot description, xacro)
@@ -175,4 +175,37 @@
       <child link="${prefix}tool0" />
     </joint>
+    <!-- Camera -->
+    <link name="camera_mount">
+    <visual>
+        <geometry>
+            <mesh filename="package://system/database/meshes/camera_mount.stl"
+                scale="1 1 1"/>
+        </geometry>
+        <material name="ABS" >
+            <color rgba="0.5 0.5 0.5 1.0" />
+            </material>
+        </visual>
+    </link>
+    <link name="camera_base">
+    <visual>
+        <geometry>
+            <mesh filename="package://system/database/meshes/d415.stl"
+                scale="1 1 1"/>
+        </geometry>
+        <material name="ABS" >
+            <color rgba="0.5 0.5 0.5 1.0" />
+            </material>
+        </visual>
+    </link>
+    <joint type="fixed" name="mount_joint">
+        <origin xyz="0 0 0" rpy="0 0 0"/>
+        <parent link="${prefix}tool0"/>
+        <child link="camera_mount"/>
+    </joint>
+    <joint type="fixed" name="camera_joint">
+        <origin xyz="-0.0145 0 0.0385" rpy="0 0 1.57"/>
+        <parent link="camera_mount"/>
+        <child link="camera_base"/>
+    </joint>
   </xacro:macro>
 </robot>

Commit message: finished baseline results.

File: src/deps/abb/abb_irb2600_support/urdf/irb2600_12_165_macro.xacro (robot description, xacro)
@@ -117,5 +117,5 @@
       <child link="${prefix}link_1" />
       <axis xyz="0 0 1" />
-      <limit lower="-3.14159" upper="3.14159" effort="0" velocity="3.054" />
+      <limit lower="-0.7" upper="3.0" effort="0" velocity="3.054" />
     </joint>
     <joint name="${prefix}joint_2" type="revolute">
@@ -138,5 +138,5 @@
       <child link="${prefix}link_4" />
       <axis xyz="1 0 0" />
-      <limit lower="-1.8" upper="5.23" effort="0" velocity="6.283" />
+      <limit lower="1.4" upper="5.0" effort="0" velocity="6.283" />
     </joint>
     <joint name="${prefix}joint_5" type="revolute">
